File: Op Amp rail splitter/Op Amp rail splitter.kicad_pcb (KiCad board)
At the start: 2 copper layers, 52.1 x 32.6 mm, 12 parts, among them J1 Vin, J2 Vout, Q1 BC547, Q2 BC557, U1 LM358

Commit message: Add DAC
Parts:
- added J3: Vout, Connector_PinHeader_2.54mm:PinHeader_1x03_P2.54mm_Vertical, F.Cu at (112.5, 109.5)
- moved J2 2.00 mm to (108.5, 109.5)
Routing:
- net /VGnd: track 43.4 -> 47.9 mm
- net VCC: track 95.7 -> 97.6 mm
Other:
- board size 52.1 x 32.6 mm -> 53.4 x 32.6 mm
