File: Teensy 9V level shifter/Teensy 9V level shifter.kicad_sch (KiCad schematic)
At the start: 47 parts, among them J1 PSU, J10 VGG, J2 TeensyL, J3 CLK, J4 ¬CLK, J5 TeensyR, J6 TeensyL1, J7 TeensyR1, J8 PSU, J9 VCA_CV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

Commit message: Strin Maschine - first revision before review
Parts:
- U6: footprint Package_TO_SOT_SMD:SOT-223-6 -> TO170P1066X482X1572-5
Other:
- moved on the sheet: C10, R12, R13

Commit message: String Maschine controller - fix broken symbols
Parts:
- removed U6: MCP1826-ADJE/AT, TO170P1066X482X1572-5, symbol mcp1826-adj:MCP1826-ADJE/AT
- added R15, R16, R17, R18: 1k, Resistor_SMD:R_0603_1608Metric_Pad0.98x0.95mm_HandSolder, symbol Device:R_Small
- added U6: MCP1826-ADJ, Package_TO_SOT_SMD:SOT-223-6, symbol custom:MCP1826-ADJ
- R10, R11, R8, R9: value 5.6k -> 10k
Connections:
- net +5V: now also U6.1 (¬SHDN), U6.2 (Vin)
- net 4.65V: now also U6.4 (Vout); no longer C10.1
- net GND: now also U6.6 (PAD); no longer J10.1 (Pin_1)
- net at R10.2, U3.8: now also R17.1; no longer J9.3 (Pin_3)
- net at R8.2, U3.1: now also R15.1; no longer J9.1 (Pin_1)
- net at R12.2, R13.1: now also U6.5 (Adj)
- net at R9.2, U3.7: now also R16.1; no longer J9.2 (Pin_2)
- net at R11.2, U3.14: now also R18.1; no longer J9.4 (Pin_4)
- new net: C10.1, J10.1 (Pin_1), U6.3 (GND)
- new net: J9.1 (Pin_1), R15.2
- new net: J9.4 (Pin_4), R18.2
- new net: J9.3 (Pin_3), R17.2
- new net: J9.2 (Pin_2), R16.2
Other:
- note added: "VCA CV outputs are scaled to -0.8 to 3.3 V (assuming 5k CV input resistance) to get >+20 to -100dB gain from VCA respectively The 1k resistors are to create a filter with a cap at CV in. See spice simulation and the voice schematic for reference."
- note removed: "VCA CV outputs are scaled to -0.64 to 3.26 V to get +20 to -100dB gain from VCA respectively"
- moved on the sheet: C10, C9, J10, J9, R14, U1A, U1B, U1C, U1D, U1E, U1F, U2A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

Commit message: String Maschine - Add simulations and add VCA for controlling the feedback loop
Parts:
- added R19: 1k, Resistor_SMD:R_0603_1608Metric_Pad0.98x0.95mm_HandSolder, symbol Device:R_Small
- R1: value 1k -> 250
- R10, R11, R8, R9: value 10k -> 20k
- R2: value 5.6k -> 12k
- R3: value 4.7k -> 15k
- TP6: value 1.145V -> 1.4V
Connections:
- net 2V5: now also R19.1
- net 4.65V: now also C10.1
- net GND: now also J10.1 (Pin_1), U6.3 (GND), R19.2
- net at TP4.1, U4.6 (VOUTC): now also R6.1; no longer U3.10 (+)
- net at TP2.1, U4.4 (VOUTA): now also R4.1; no longer U3.3 (+)
- net at TP5.1, U4.5 (VOUTB): now also R5.1; no longer U3.5 (+)
- net at U4.7 (VOUTD): now also R7.1; no longer U3.12 (+)
- removed net 1.145V: R2.2, R3.1, R4.1, R5.1, R6.1, R7.1, TP6.1
- new net 1.4V: R2.2, R3.1, TP6.1, U3.10 (+), U3.12 (+), U3.3 (+), U3.5 (+)
Other:
- moved on the sheet: C10, C8, J9, R1, R10, R11, R15, R16, R17, R18, R4, R5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
