File: String Maschine/String Maschine.kicad_sch (KiCad schematic)
At the start: 67 parts, among them J1 Vin, J2 VGG, J3 VOut, J4 Vin, J5 CTLS, J6 VGG, SW1 FBACK, SW2 NOISE, SW3 FBACK, SW4 SW_SPDT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

Commit message: String Maschine - finish voice board
Parts:
- removed J5: CTLS, Connector_PinHeader_2.54mm:PinHeader_1x04_P2.54mm_Vertical, symbol Connector:Conn_01x04_Female
- added J5: CTLS, Connector_PinHeader_2.54mm:PinHeader_1x05_P2.54mm_Vertical, symbol Connector:Conn_01x05_Female
- C1, C10, C11, C12, C13, C14, C15, C16, C18, C7: footprint Capacitor_THT:C_Rect_L7.0mm_W4.5mm_P5.00mm -> Capacitor_THT:C_Rect_L7.0mm_W3.5mm_P5.00mm
- C17, C2, C4, C6: footprint Capacitor_THT:C_Rect_L7.0mm_W4.5mm_P5.00mm -> Capacitor_THT:C_Disc_D5.0mm_W2.5mm_P5.00mm
- C3, C5: footprint Capacitor_THT:C_Rect_L7.0mm_W4.5mm_P5.00mm -> Capacitor_THT:C_Rect_L7.0mm_W2.5mm_P5.00mm
- D1, D2: footprint Diode_THT:D_DO-41_SOD81_P10.16mm_Horizontal -> Diode_THT:D_DO-41_SOD81_P7.62mm_Horizontal
- IN1: renamed from SW4; value SW_SPDT -> J_IN; footprint (none) -> Connector_PinHeader_2.54mm:PinHeader_1x03_P2.54mm_Vertical
- J6: value VGG -> EXTIN
- SW1: value FBACK -> JFOUT
- SW2: value NOISE -> EN_IN
- SW3: value FBACK -> JFIN
- TP12: value CVN -> CVVCA
- renumbered VNOISE1 to IN_VOL1
Connections:
- net CP1: now also J5.4 (Pin_4)
- net CP2: now also J5.5 (Pin_5)
- net CVF: now also U1.11, J5.2 (Pin_2); no longer U1.3
- net CVN: now also U1.3, J5.1 (Pin_1); no longer U1.14
- net CVVCA: now also U1.14, J5.3 (Pin_3); no longer U1.11
- net at C5.1, R8.1, R9.2: now also U2.8; no longer U2.1
- net at R1.1, R14.1: now also U1.15; no longer U1.10
- net at R17.2, U2.13 (-): now also U1.13; no longer U1.12
- net at C9.1, R20.2, R5.1: now also U2.1; no longer U2.8
- net at R4.1, R5.2, SW2.2 (B): now also U2.2 (-); no longer U2.9 (-)
- net at SW2.1 (A): now also U1.4; no longer U1.13
- net at R2.1, R3.1, TP1.1: now also U1.2; no longer U1.15
- net at R15.1, R16.2, R9.1: now also U1.10; no longer U1.2
- new net: C5.2, U1.12, U2.9 (-)
Other:
- moved on the sheet: U1A, U1C, U1D, U2A, U2C
